Commit message: Added path planning module

File: hsi/envs/urdf/arial_vehicle_collision_free.urdf (robot description, URDF)
Before this commit: robot environment, 1 links, 0 joints
Links:
- link base_link: geometry visual sphere radius=0.75

File: hsi/envs/urdf/environment_collision_free.urdf (robot description, URDF)
Before this commit: robot environment, 1 links, 0 joints
Links:
- link buildings: mass 1 -> 0; geometry visual mesh filename=meshes/test.obj

File: hsi/envs/urdf/ground_vehicle.urdf (robot description, URDF)
Before this commit: robot environment, 1 links, 0 joints
Links:
- link base_link: geometry collision box size=0.75 0.75 0.75; visual box size=0.75 0.75 0.75

File: hsi/envs/urdf/ground_vehicle_collision_free.urdf (robot description, URDF)
Before this commit: robot environment, 1 links, 0 joints
Links:
- link base_link: geometry visual box size=1 1 1
